File: PCB/MaxRam.kicad_pcb (KiCad board)
At the start: 2 copper layers, 76.2 x 43.2 mm, 16 parts, among them J1 CONN_01X14, J3 CONN_02X05, J4 GS3, J5 GS3, J6 CONN_01X14, J7 CONN_01X02, J8 CONN_01X08, U1 AS6C4008-55SIN, U2 SST39SF040, U3 ATF1502PLCC44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

Commit message: Post up Issue A as sent to OSH Park
Routing:
- net /A11: track 71.8 -> 73.3 mm
- net +5V: track 128.7 -> 129.3 mm
- net /A9: track 75.4 -> 76.0 mm
- net /nWE: track 50.0 -> 49.4 mm
- net /A8: track 79.4 -> 78.9 mm
- net /A12: vias 4 -> 3
Other:
- outline, holes or cut-outs redrawn
- net class Default: via_dia 0.6 -> 0.6858
- net class Power: via_dia 0.6 -> 0.6858
- board text added: "AT28C256"
- board text added: "or"
